File: Joystick rate and LCD Circuit tinkercad.brd (EAGLE design)
At the start: 68.6 x 53.3 mm, 11 parts

Commit message: Update Joystick rate and LCD Circuit tinkercad.brd
Connections:
- new net N$15: R1.1, U1.6
- new net N$16: R3.2, S1.1, U1.7
- new net N$17: R2.1, U1.13
